Commit message: Edit urdf

File: resources/robots/x1/urdf/x1.urdf (robot description, URDF)
Before this commit: robot x1, 58 links, 57 joints
Links:
- link arm_l_wrist_a_ball: geometry visual mesh filename=package://x1/meshes/arm_r_wrist_a_ball.STL
- link arm_l_wrist_a_loop: geometry visual mesh filename=package://x1/meshes/arm_r_wrist_a_loop.STL
- link arm_l_wrist_b_ball: geometry visual mesh filename=package://x1/meshes/arm_r_wrist_b_ball.STL
- link arm_l_wrist_b_loop: geometry visual mesh filename=package://x1/meshes/arm_r_wrist_b_loop.STL
- link arm_l_wrist_motor_a_link: geometry visual mesh filename=package://x1/meshes/arm_r_wrist_motor_a_link.STL
- link arm_l_wrist_motor_b_link: geometry visual mesh filename=package://x1/meshes/arm_r_wrist_motor_b_link.STL
- link arm_r_wrist_a_ball: geometry visual mesh filename=package://x1/meshes/arm_r_wrist_a_ball.STL
- link arm_r_wrist_a_loop: geometry visual mesh filename=package://x1/meshes/arm_r_wrist_a_loop.STL
- link arm_r_wrist_b_ball: geometry visual mesh filename=package://x1/meshes/arm_r_wrist_b_ball.STL
- link arm_r_wrist_b_loop: geometry visual mesh filename=package://x1/meshes/arm_r_wrist_b_loop.STL
- link arm_r_wrist_motor_a_link: geometry visual mesh filename=package://x1/meshes/arm_r_wrist_motor_a_link.STL
- link arm_r_wrist_motor_b_link: geometry visual mesh filename=package://x1/meshes/arm_r_wrist_motor_b_link.STL
- link base_link: geometry collision mesh filename=package://x1/meshes/base_link_simple.STL; visual mesh filename=package://x1/meshes/base_link_simple.STL
- link left_ankle_pitch: geometry visual mesh filename=package://x1/meshes/left_ankle_pitch.STL
- link left_ankle_roll: geometry collision mesh filename=package://x1/meshes/left_ankle_roll.STL; visual mesh filename=package://x1/meshes/left_ankle_roll.STL
- link left_elbow_pitch: geometry visual mesh filename=package://x1/meshes/left_elbow_pitch.STL
- link left_elbow_yaw: geometry visual mesh filename=package://x1/meshes/left_elbow_yaw.STL
- link left_hip_pitch: geometry visual mesh filename=package://x1/meshes/left_hip_pitch.STL
- link left_hip_roll: geometry visual mesh filename=package://x1/meshes/left_hip_roll.STL
- link left_hip_yaw: geometry visual mesh filename=package://x1/meshes/left_hip_yaw.STL
- link left_knee_pitch: geometry visual mesh filename=package://x1/meshes/left_knee_pitch.STL
- link left_shoulder_pitch: geometry visual mesh filename=package://x1/meshes/left_shoulder_pitch.STL
- link left_shoulder_roll: geometry visual mesh filename=package://x1/meshes/left_shoulder_roll.STL
- link left_shoulder_yaw: geometry visual mesh filename=package://x1/meshes/left_shoulder_yaw.STL
- link left_wrist_pitch: geometry visual mesh filename=package://x1/meshes/left_wrist_pitch.STL
- link leg_l_toe_a_ball: geometry visual mesh filename=package://x1/meshes/leg_l_toe_a_ball.STL
- link leg_l_toe_a_link: geometry visual mesh filename=package://x1/meshes/leg_l_toe_a_link.STL
- link leg_l_toe_a_loop: geometry visual mesh filename=package://x1/meshes/leg_l_toe_a_loop.STL
- link leg_l_toe_b_ball: geometry visual mesh filename=package://x1/meshes/leg_l_toe_b_ball.STL
- link leg_l_toe_b_link: geometry visual mesh filename=package://x1/meshes/leg_l_toe_b_link.STL
- link leg_l_toe_b_loop: geometry visual mesh filename=package://x1/meshes/leg_l_toe_b_loop.STL
- link leg_r_toe_a_ball: geometry visual mesh filename=package://x1/meshes/leg_r_toe_a_ball.STL
- link leg_r_toe_a_link: geometry visual mesh filename=package://x1/meshes/leg_r_toe_a_link.STL
- link leg_r_toe_a_loop: geometry visual mesh filename=package://x1/meshes/leg_r_toe_a_loop.STL
- link leg_r_toe_b_ball: geometry visual mesh filename=package://x1/meshes/leg_r_toe_b_ball.STL
- link leg_r_toe_b_link: geometry visual mesh filename=package://x1/meshes/leg_r_toe_b_link.STL
- link leg_r_toe_b_loop: geometry visual mesh filename=package://x1/meshes/leg_r_toe_b_loop.STL
- link lumber_pitch: geometry visual mesh filename=package://x1/meshes/lumber_pitch.STL
- link lumber_roll: geometry visual mesh filename=package://x1/meshes/lumber_roll.STL
- link lumber_yaw: geometry visual mesh filename=package://x1/meshes/lumber_yaw.STL
- link right_ankle_pitch: geometry visual mesh filename=package://x1/meshes/right_ankle_pitch.STL
- link right_ankle_roll: geometry collision mesh filename=package://x1/meshes/right_ankle_roll.STL; visual mesh filename=package://x1/meshes/right_ankle_roll.STL
- link right_elbow_pitch: geometry visual mesh filename=package://x1/meshes/right_elbow_pitch.STL
- link right_elbow_yaw: geometry visual mesh filename=package://x1/meshes/right_elbow_yaw.STL
- link right_hip_pitch: geometry visual mesh filename=package://x1/meshes/right_hip_pitch.STL
- link right_hip_roll: geometry visual mesh filename=package://x1/meshes/right_hip_roll.STL
- link right_hip_yaw: geometry visual mesh filename=package://x1/meshes/right_hip_yaw.STL
- link right_knee_pitch: geometry visual mesh filename=package://x1/meshes/right_knee_pitch.STL
- link right_shoulder_pitch: geometry visual mesh filename=package://x1/meshes/right_shoulder_pitch.STL
- link right_shoulder_roll: geometry visual mesh filename=package://x1/meshes/right_shoulder_roll.STL
- link right_shoulder_yaw: geometry visual mesh filename=package://x1/meshes/right_shoulder_yaw.STL
- link right_wrist_pitch: geometry visual mesh filename=package://x1/meshes/right_wrist_pitch.STL
- link waist_motor_a_ball: geometry visual mesh filename=package://x1/meshes/waist_motor_a_ball.STL
- link waist_motor_a_link: geometry visual mesh filename=package://x1/meshes/waist_motor_a_link.STL
- link waist_motor_a_loop: geometry visual mesh filename=package://x1/meshes/waist_motor_a_loop.STL
- link waist_motor_b_ball: geometry visual mesh filename=package://x1/meshes/waist_motor_b_ball.STL
- link waist_motor_b_link: geometry visual mesh filename=package://x1/meshes/waist_motor_b_link.STL
- link waist_motor_b_loop: geometry visual mesh filename=package://x1/meshes/waist_motor_b_loop.STL
Joints:
- joint left_elbow_pitch_joint: type fixed -> revolute
- joint left_elbow_yaw_joint: type fixed -> revolute
- joint left_shoulder_pitch_joint: type fixed -> revolute
- joint left_shoulder_roll_joint: type fixed -> revolute
- joint left_shoulder_yaw_joint: type fixed -> revolute
- joint left_wrist_pitch_joint: type fixed -> revolute
- joint lumber_pitch_joint: type fixed -> revolute
- joint lumber_roll_joint: type fixed -> revolute
- joint lumber_yaw_joint: type fixed -> revolute
- joint right_elbow_pitch_joint: type fixed -> revolute
- joint right_elbow_yaw_joint: type fixed -> revolute
- joint right_shoulder_pitch_joint: type fixed -> revolute
- joint right_shoulder_roll_joint: type fixed -> revolute
- joint right_shoulder_yaw_joint: type fixed -> revolute
- joint right_wrist_pitch_joint: type fixed -> revolute

Commit message: Fix lumber_roll_joint and lumber_pitch_joint

File: resources/robots/x1/urdf/x1.urdf (robot description, URDF)
Before this commit: robot x1, 58 links, 57 joints
Joints:
- joint lumber_pitch_joint: type revolute -> fixed
- joint lumber_roll_joint: type revolute -> fixed

Commit message: Fix joint limits

File: resources/robots/x1/urdf/x1.urdf (robot description, URDF)
Before this commit: robot x1, 58 links, 57 joints
Joints:
- joint left_elbow_pitch_joint: limit lower=-3.14 upper=3.14 effort=0 velocity=0 -> lower=0.0 upper=1.7 effort=0 velocity=0
- joint left_shoulder_roll_joint: limit lower=-3.14 upper=3.14 effort=0 velocity=0 -> lower=-3.14 upper=0.0 effort=0 velocity=0
- joint right_elbow_pitch_joint: limit lower=-3.14 upper=3.14 effort=0 velocity=0 -> lower=0.0 upper=1.7 effort=0 velocity=0
- joint right_shoulder_roll_joint: limit lower=-3.14 upper=3.14 effort=0 velocity=0 -> lower=-3.14 upper=0.0 effort=0 velocity=0

Commit message: Update joint limits

File: resources/robots/x1/urdf/x1.urdf (robot description, URDF)
Before this commit: robot x1, 58 links, 57 joints
Joints:
- joint left_elbow_yaw_joint: limit lower=-3.14 upper=3.14 effort=0 velocity=0 -> lower=-0.8 upper=0.8 effort=0 velocity=0
- joint left_shoulder_pitch_joint: limit lower=-3.14 upper=3.14 effort=0 velocity=0 -> lower=-2.2 upper=0.0 effort=0 velocity=0
- joint left_shoulder_roll_joint: limit lower=-3.14 upper=0.0 effort=0 velocity=0 -> lower=-2.3 upper=0.0 effort=0 velocity=0
- joint left_shoulder_yaw_joint: limit lower=-3.14 upper=3.14 effort=0 velocity=0 -> lower=-0.5 upper=0.5 effort=0 velocity=0
- joint left_wrist_pitch_joint: limit lower=-3.14 upper=3.14 effort=0 velocity=0 -> lower=0.0 upper=0.0 effort=0 velocity=0
- joint lumber_pitch_joint: limit lower=-3.14 upper=3.14 effort=0 velocity=0 -> lower=0.0 upper=0.2 effort=0 velocity=0; type fixed -> revolute
- joint lumber_yaw_joint: limit lower=-3.14 upper=3.14 effort=0 velocity=0 -> lower=-0.8 upper=0.8 effort=0 velocity=0
- joint right_elbow_yaw_joint: limit lower=-3.14 upper=3.14 effort=0 velocity=0 -> lower=-0.8 upper=0.8 effort=0 velocity=0
- joint right_shoulder_pitch_joint: limit lower=-3.14 upper=3.14 effort=0 velocity=0 -> lower=-2.2 upper=0.0 effort=0 velocity=0
- joint right_shoulder_roll_joint: limit lower=-3.14 upper=0.0 effort=0 velocity=0 -> lower=-2.3 upper=0.0 effort=0 velocity=0
- joint right_shoulder_yaw_joint: limit lower=-3.14 upper=3.14 effort=0 velocity=0 -> lower=-0.5 upper=0.5 effort=0 velocity=0
- joint right_wrist_pitch_joint: limit lower=-3.14 upper=3.14 effort=0 velocity=0 -> lower=0.0 upper=0.0 effort=0 velocity=0

Commit message: Disable lumber_pitch_joint

File: resources/robots/x1/urdf/x1.urdf (robot description, URDF)
Before this commit: robot x1, 58 links, 57 joints
Joints:
- joint lumber_pitch_joint: limit lower=0.0 upper=0.2 effort=0 velocity=0 -> lower=-3.14 upper=3.14 effort=0 velocity=0; type revolute -> fixed

Commit message: Disable lumber_yaw_joint first

File: resources/robots/x1/urdf/x1.urdf (robot description, URDF)
Before this commit: robot x1, 58 links, 57 joints
Joints:
- joint lumber_yaw_joint: limit lower=-0.8 upper=0.8 effort=0 velocity=0 -> lower=-3.14 upper=3.14 effort=0 velocity=0; type revolute -> fixed

Commit message: Increase joint limits

File: resources/robots/x1/urdf/x1.urdf (robot description, URDF)
Before this commit: robot x1, 58 links, 57 joints
Joints:
- joint left_elbow_yaw_joint: limit lower=-0.8 upper=0.8 effort=0 velocity=0 -> lower=-1.2 upper=1.2 effort=0 velocity=0
- joint left_shoulder_pitch_joint: limit lower=-2.2 upper=0.0 effort=0 velocity=0 -> lower=-2.6 upper=0.0 effort=0 velocity=0
- joint left_shoulder_roll_joint: limit lower=-2.3 upper=0.0 effort=0 velocity=0 -> lower=-2.7 upper=0.0 effort=0 velocity=0
- joint left_shoulder_yaw_joint: limit lower=-0.5 upper=0.5 effort=0 velocity=0 -> lower=-0.9 upper=0.9 effort=0 velocity=0
- joint right_elbow_yaw_joint: limit lower=-0.8 upper=0.8 effort=0 velocity=0 -> lower=-1.2 upper=1.2 effort=0 velocity=0
- joint right_shoulder_pitch_joint: limit lower=-2.2 upper=0.0 effort=0 velocity=0 -> lower=-2.6 upper=0.0 effort=0 velocity=0
- joint right_shoulder_roll_joint: limit lower=-2.3 upper=0.0 effort=0 velocity=0 -> lower=-2.7 upper=0.0 effort=0 velocity=0
- joint right_shoulder_yaw_joint: limit lower=-0.5 upper=0.5 effort=0 velocity=0 -> lower=-0.9 upper=0.9 effort=0 velocity=0
